File: flat_memory_32k.kicad_pcb (KiCad board)
At the start: 2 copper layers, 85 x 65 mm, 41 parts, among them X1 Power, X2 Address, X3 Data, X4 Mode, X5 Control, X6 Clock

Commit message: Update
Parts:
- removed C5: 1u, Capacitor_Tantalum_SMD:CP_EIA-3216-18_Kemet-A_Pad1.58x1.35mm_HandSolder
- added C19: 1u, Capacitor_Tantalum_SMD:CP_EIA-3216-18_Kemet-A_Pad1.58x1.35mm_HandSolder, B.Cu at (118.6, 84.3)
- added C8: 1u, Capacitor_Tantalum_SMD:CP_EIA-3216-18_Kemet-A_Pad1.58x1.35mm_HandSolder, B.Cu at (85.9, 104.5)
- C16: value 1u -> 100n; footprint Capacitor_Tantalum_SMD:CP_EIA-3216-18_Kemet-A_Pad1.58x1.35mm_HandSolder -> Capacitor_SMD:C_0805_2012Metric_Pad1.18x1.45mm_HandSolder
- moved C7 49.1 mm to (88.8, 102.4)
- moved C13 37.3 mm to (145.0, 90.9)
- moved C17 24.0 mm to (106.6, 84.3)
- moved C14 24.0 mm to (108.8, 81.9)
- moved C1 20.7 mm to (106.3, 101.2), turned to 90 degrees
- moved C2 19.7 mm to (108.4, 101.6), turned to 90 degrees
- moved C6 15.4 mm to (137.9, 104.5), turned to 180 degrees
- moved C4 14.4 mm to (122.8, 101.6)
- moved C3 14.3 mm to (120.6, 101.2)
- moved C16 14.3 mm to (120.7, 81.9), turned to 90 degrees
- moved C18 12.1 mm to (130.6, 84.3)
- moved C15 12.1 mm to (132.8, 81.9)
Connections:
- C13 pad 1: +5 -> GND
- C13 pad 2: GND -> Net-(DD9-E3)
Routing:
- net Net-(DD9-E3): track 2.32 -> 4.25 mm
- net GND: vias 256 -> 306
Other:
- board text added: "DB6"

Commit message: Fix silk
Other:
- board text added: "R2AKT.467522.002"
- board text removed: "R2AKT.467562.002"
Changed lines of the file:
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@@
 		(date "2026-03-11")
 		(company "R2AKT")
-		(comment 1 "R2AKT.467562.002")
+		(comment 1 "R2AKT.467522.002")
 		(comment 2 "R2AKT")
 	)
@@
 		)
 	)
-	(gr_text "R2AKT.467562.002"
+	(gr_text "R2AKT.467522.002"
 		(at 89.093428 99.6696 0)
 		(layer "F.SilkS")
