File: flat_memory_32k.kicad_sch (KiCad schematic)
At the start: 40 parts, among them X1 Power, X2 Address, X3 Data, X4 Mode, X5 Control, X6 Clock

Commit message: Update
Parts:
- removed C16, C8: 1u, Capacitor_Tantalum_SMD:CP_EIA-3216-18_Kemet-A_Pad1.58x1.35mm_HandSolder, symbol Device:C_Polarized
- added C16: 100n, Capacitor_SMD:C_0805_2012Metric_Pad1.18x1.45mm_HandSolder, symbol Device:C
- added C19, C5: 1u, Capacitor_Tantalum_SMD:CP_EIA-3216-18_Kemet-A_Pad1.58x1.35mm_HandSolder, symbol Device:C_Polarized
- renumbered C5 to C8
Connections:
- net +5: now also C16.1, C19.1, C5.1; no longer C13.1
- net GND: now also C13.1, C16.2, C19.2, C5.2; no longer C13.2
- net at DD9.6 (E3), R3.1: now also C13.2
- net INTE renamed ~{WRQ}
- net Single_BCLK renamed F2TTL
- net Single_OSC_TTL renamed OSC_TTL
Other:
- moved on the sheet: C8
